Commit message: About to verify distances using selector tool

File: src/xarm_description/urdf/lite6.urdf (robot description, URDF)
Before this commit: robot lite6, 11 links, 10 joints
Joints:
- joint left_finger_joint: origin xyz=0.0 0.021 0.0817 rpy=0 0 0 -> xyz=0.0 0.023 0.0817 rpy=0 0 0
- joint right_finger_joint: origin xyz=0.0 -0.021 0.0817 rpy=0 0 0 -> xyz=0.0 -0.023 0.0817 rpy=0 0 0

Commit message: Added joint between coupler and gripper base

File: src/xarm_description/urdf/lite6.urdf (robot description, URDF)
Before this commit: robot lite6, 11 links, 10 joints
Links:
- added link omx_gripper_joint, mass 0.001; collision box size=0.001 0.001 0.001; visual box size=0.001 0.001 0.001
Joints:
- added joint omx_gripper_fixed_joint: type fixed, parent lite6_gripper_link, child omx_gripper_joint, origin xyz=0 0 0 rpy=0 0 0
- joint joint3: origin xyz=0.2 0 0 rpy=-3.1416 0 1.5708 -> xyz=0.2 0 0 rpy=-3.1416 0 0
